Commit message: checkpoint: slam_toolbox started mapping

File: ros_park_n_pi/src/raspbotv2_bringup/urdf/RaspbotV2.urdf (robot description, URDF)
Before this commit: robot RaspbotV2.urdf, 13 links, 12 joints
Links:
- added link base_footprint
- link arm1_Link: geometry visual mesh filename=package://raspbotv2_bringup/meshes/arm1_Link.stl
- link arm2_Link: geometry visual mesh filename=package://raspbotv2_bringup/meshes/arm2_Link.stl
- link base_link: geometry collision box size=0.11 0.19 0.09; visual mesh filename=package://raspbotv2_bringup/meshes/base_Link.stl
- link l1_Link: geometry collision cylinder length=0.03 radius=0.029; visual mesh filename=package://raspbotv2_bringup/meshes/l1_Link.stl
- link l2_Link: geometry collision cylinder length=0.03 radius=0.029; visual mesh filename=package://raspbotv2_bringup/meshes/l2_Link.stl
- link r1_Link: geometry collision cylinder length=0.03 radius=0.029; visual mesh filename=package://raspbotv2_bringup/meshes/r1_Link.stl
- link r2_Link: geometry collision cylinder length=0.03 radius=0.029; visual mesh filename=package://raspbotv2_bringup/meshes/r2_Link.stl
Joints:
- added joint base_footprint_joint: type fixed, parent base_link, child base_footprint, origin xyz=0 0 0 rpy=0 0 0
